File: DirtyMirror.kicad_pcb (KiCad board)
At the start: 2 copper layers, 82 x 49 mm, 76 parts, among them J101 PWR, J102 ScopeGroundLoop, SW101 SW_SPDT, U101 TL074, U102 TL074

Commit message: rev3 minor tweaks
Parts:
- added R137: 100k, Resistor_SMD:R_0805_2012Metric, B.Cu at (26.1, 82.9)
- added R138: 47k, Resistor_SMD:R_0805_2012Metric, B.Cu at (16.1, 83.0)
- added R139: 100k, Resistor_SMD:R_0805_2012Metric, B.Cu at (21.8, 61.6)
- added TP112: SKEW, TestPoint:TestPoint_THTPad_D2.0mm_Drill1.0mm_VAL, F.Cu at (12.2, 80.1)
- moved R106 50.7 mm to (66.0, 74.0), turned to 180 degrees
- moved TP103 42.3 mm to (81.7, 79.2)
- moved R107 41.7 mm to (66.0, 70.8), turned to 180 degrees
- moved TP101 1.20 mm to (21.8, 57.9), turned to 180 degrees
- moved R122 0.72 mm to (23.1, 66.3)
Connections:
- R106 pad 2: Net-(R106-Pad2) -> /LoThresh
- RV101 pad 1: Net-(R106-Pad2) -> Net-(R138-Pad1)
- RV101 pad 2: /LoThresh -> /vSkew
- RV101 pad 3: /LoThresh -> Net-(R137-Pad2)
Routing:
- net /vSkew: track 0.00 -> 36.4 mm, vias 0 -> 1
- net /LoThresh: track 54.3 -> 29.8 mm
- net +9V: track 91.4 -> 111.3 mm, vias 1 -> 2
- net Net-(U101D--): track 6.30 -> 13.4 mm
- net Net-(R108-Pad2): track 7.09 -> 11.2 mm
- net GND: track 0.00 -> 3.57 mm, vias 0 -> 1
- net /Bias: track 96.8 -> 99.6 mm
- net Net-(R137-Pad2): track 0.00 -> 2.74 mm
- net Net-(R106-Pad2): track 2.74 -> 0.00 mm
- net Net-(R138-Pad1): track 0.00 -> 2.64 mm
- net /Gtr_gain: track 96.8 -> 98.8 mm
- net /LoRect: track 44.0 -> 45.6 mm
Other:
- board text added: "Rev 3- Jan 2025 Hayden Setlik"
- board text removed: "Rev 2- Jan 2025 Hayden Setlik"

Commit message: silkscreen and spacing niceities
Parts:
- moved J102 33.4 mm to (36.6, 82.7)
- moved TP111 18.0 mm to (63.4, 49.1)
- moved TP102 10.8 mm to (59.1, 87.2), turned to 180 degrees
- moved R128 9.64 mm to (64.3, 88.2)
- moved R137 5.17 mm to (30.5, 85.7)
- moved R138 4.77 mm to (12.2, 85.6)
- moved TP109 4.15 mm to (31.1, 77.0)
- moved TP110 3.60 mm to (59.3, 46.3)
- moved R132 1.25 mm to (54.0, 47.1)
- moved C106 1.21 mm to (73.8, 45.2)
- moved R139 0.45 mm to (21.8, 62.0)
Routing:
- net /Fold: track 51.4 -> 68.9 mm, vias 0 -> 1
- net Net-(R128-Pad1): track 2.77 -> 12.9 mm
- net FX_OUT: track 27.6 -> 18.6 mm
- net /Clip: track 22.2 -> 26.1 mm
- net /Gtr_gain: track 98.8 -> 101.8 mm
- net Net-(C106-Pad2): track 23.0 -> 24.7 mm
- net Net-(R137-Pad2): track 2.74 -> 4.38 mm
- net Net-(R138-Pad1): track 2.64 -> 4.02 mm
- net +9V: track 111.3 -> 110.1 mm
- net /LoRect: track 45.6 -> 46.3 mm
- net Net-(R132-Pad2): track 5.33 -> 5.89 mm
- net /Bias: track 99.6 -> 99.1 mm
Other:
- board text added: "Gain"
- board text added: "Shape"
- board text added: "Skew"
- board text added: "Tone"
- board text added: "Volume"
