File: DirtyMirror.kicad_pcb (KiCad board)
At the start: 2 copper layers, 82 x 49 mm, 76 parts, among them J101 PWR, J102 ScopeGroundLoop, SW101 SW_SPDT, U101 TL074, U102 TL074

Commit message: component values
Parts:
- R102: value 2k2 -> 10k
- R132, R134: value 4k7 -> 47k
- RV102: value 10k -> 100k
- RV103: value 10kB -> 100kB
Changed lines of the file:
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@@
 			)
 		)
-		(property "Value" "10k"
+		(property "Value" "100k"
 			(at 4.9 -24.3 180)
 			(layer "F.Fab")
@@
 			)
 		)
-		(property "Value" "10kB"
+		(property "Value" "100kB"
 			(at 4.9 -24.3 180)
 			(layer "F.Fab")
@@
 			)
 		)
-		(property "Value" "4k7"
+		(property "Value" "47k"
 			(at 0 -1.65 90)
 			(layer "B.Fab")
@@
 			)
 		)
-		(property "Value" "4k7"
+		(property "Value" "47k"
 			(at 0 -1.65 90)
 			(layer "B.Fab")
@@
 			)
 		)
-		(property "Value" "2k2"
+		(property "Value" "10k"
 			(at 0 -1.65 90)
 			(layer "B.Fab")

Commit message: changed schematic to reflect bodging
Parts:
- C107: value 100n -> 10n
- R106: value 51k -> 510k
- R107: value 47k -> 470k
- R124: value 1k8 -> 12k
- R130: value 33k -> 39k
- RV101, RV104: value 10kB -> 100kB
- RV102: value 100k -> 100kB
Changed lines of the file:
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@@
 			)
 		)
-		(property "Value" "10kB"
+		(property "Value" "100kB"
 			(at 4.9 -24.3 180)
 			(layer "F.Fab")
@@
 			)
 		)
-		(property "Value" "100k"
+		(property "Value" "100kB"
 			(at 4.9 -24.3 180)
 			(layer "F.Fab")
@@
 			)
 		)
-		(property "Value" "10kB"
+		(property "Value" "100kB"
 			(at 4.9 -24.3 180)
 			(layer "F.Fab")
@@
 			)
 		)
-		(property "Value" "100n"
+		(property "Value" "10n"
 			(at 0 -1.679999 90)
 			(layer "B.Fab")
@@
 			)
 		)
-		(property "Value" "51k"
+		(property "Value" "510k"
 			(at 0 -1.65 90)
 			(layer "B.Fab")
@@
 			)
 		)
-		(property "Value" "33k"
+		(property "Value" "39k"
 			(at 0 -1.65 0)
 			(layer "B.Fab")
@@
 			)
 		)
-		(property "Value" "1k8"
+		(property "Value" "12k"
 			(at 0 -1.65 90)
 			(layer "B.Fab")
@@
 			)
 		)
-		(property "Value" "47k"
+		(property "Value" "470k"
 			(at 0 -1.65 90)
 			(layer "B.Fab")
