File: DirtyMirror.kicad_sch (KiCad schematic)
At the start: 72 parts, among them J101 PWR, J102 ScopeGroundLoop, SW101 SW_SPDT, U101 TL074, U102 TL074

Commit message: changed schematic to reflect bodging
Parts:
- removed R130: 33k, Resistor_SMD:R_0805_2012Metric, symbol Device:R_US
- removed R131: 10k, Resistor_SMD:R_0805_2012Metric, symbol Device:R_US
- C103: value 2u2 -> 470n
- C107: value 100n -> 10n
- R106: value 51k -> 510k
- R107: value 47k -> 470k
- R109: value 100k -> 39k
- R124: value 1k8 -> 12k
- RV101, RV104: value 10kB -> 100kB
- RV102: value 100k -> 100kB
Connections:
- net FxFull: now also C111.2, U101.8, U101.9 (-); no longer R136.2, U101.1
- net Gtr_gain: now also RV102.2; no longer C111.2, U101.8
- net at R122.1: now also R136.2, U101.1; no longer RV102.2
Other:
- moved on the sheet: C104, C106, C107, C108, C109, C111, D101, D102, D103, D104, R110, R111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
